Commit message: Speed up media: simplify robot meshes 28.6MB->~9MB, video posters, WebP images
- Decimate G1/Inhabit/UR5 meshes (UR5 Collada -> binary STL, same geometry frame)
- Poster frames on video tiles + modal so they never show blank; strip unused audio
- Start fetching videos/meshes earlier (600px / 400px ahead of viewport)
- Swap heavy PNG/JPG tiles for WebP (cad-7 2.0MB -> 53KB)

Co-Authored-By: Claude Opus 5.5 <noreply@anthropic.com>

File: robots/ur5/ur5.urdf (robot description, URDF)
Before this commit: robot ur5, 11 links, 10 joints
Links:
- link base_link: geometry collision mesh filename=package://ur5_description/meshes/ur5/collision/base.stl; visual mesh filename=package://ur5_description/meshes/ur5/visual/base.stl
- link forearm_link: geometry collision mesh filename=package://ur5_description/meshes/ur5/collision/forearm.stl; visual mesh filename=package://ur5_description/meshes/ur5/visual/forearm.stl
- link shoulder_link: geometry collision mesh filename=package://ur5_description/meshes/ur5/collision/shoulder.stl; visual mesh filename=package://ur5_description/meshes/ur5/visual/shoulder.stl
- link upper_arm_link: geometry collision mesh filename=package://ur5_description/meshes/ur5/collision/upperarm.stl; visual mesh filename=package://ur5_description/meshes/ur5/visual/upperarm.stl
- link wrist_1_link: geometry collision mesh filename=package://ur5_description/meshes/ur5/collision/wrist1.stl; visual mesh filename=package://ur5_description/meshes/ur5/visual/wrist1.stl
- link wrist_2_link: geometry collision mesh filename=package://ur5_description/meshes/ur5/collision/wrist2.stl; visual mesh filename=package://ur5_description/meshes/ur5/visual/wrist2.stl
- link wrist_3_link: geometry collision mesh filename=package://ur5_description/meshes/ur5/collision/wrist3.stl; visual mesh filename=package://ur5_description/meshes/ur5/visual/wrist3.stl
